Commit message: Converted code into xacro

File: install/my_robot_description/share/my_robot_description/urdf/mobile_robot.urdf (robot description, URDF)
Before this commit: robot mobile_robot, 5 links, 4 joints
Links:
- link base_link: geometry visual box size=${length} ${width} ${height}
- link left_back_wheel: geometry visual cylinder length=${wheellen} radius=${wheeldia/2}
- link left_front_wheel: geometry visual cylinder length=${wheellen} radius=${wheeldia/2}
- link right_back_wheel: geometry visual cylinder length=${wheellen} radius=${wheeldia/2}
- link right_front_wheel: geometry visual cylinder length=${wheellen} radius=${wheeldia/2}
