Commit message: Added physics for the model

File: install/my_robot_description/share/my_robot_description/urdf/mobile_robot.urdf.xacro (robot description, xacro)
@@ -1,46 +1 @@
-<?xml version="1.0"?>
-<robot name="macroed" xmlns:xacro="http://ros.org/wiki/xacro">
-  <xacro:property name="length" value="0.4" />
-  <xacro:property name="width" value="0.25" />
-  <xacro:property name="height" value="0.1" />
-  <xacro:property name="wheellen" value="0.1" />
-  <xacro:property name="wheeldia" value="0.07" />
-  <material name="blue">
-    <color rgba="0 0 0.8 1"/>
-  </material>
-  <material name="black">
-    <color rgba="0 0 0 1"/>
-  </material>
-  <material name="white">
-    <color rgba="1 1 1 1"/>
-  </material>
-   <link name="base_link">
-  <visual>
-    <geometry>
-     <box size="${length} ${width} ${height}"/>
-    </geometry>
-    <material name="blue"/>
-  </visual>
-  </link>
-  <xacro:macro name="wheel" params="name x y">
-    <link name="${name}">
-      <visual>
-        <origin xyz="0 0 0" rpy="${pi/2} 0 0" />
-        <geometry>
-          <cylinder radius="${wheeldia/2}" length="${wheellen}"/>
-        </geometry>
-        <material name="black"/>
-      </visual>
-    </link>
-     <joint name="$base_to_${name}" type="fixed">
-      <axis xyz="0 1 0" rpy="0 0 0" />
-      <parent link="base_link"/>
-      <child link="${name}"/>
-      <origin xyz="${x} ${y} -0.05" rpy="0 0 0"/>
-    </joint>
-  </xacro:macro>
-<xacro:wheel name="right_front_wheel" x="0.15" y="-0.17"/>
-<xacro:wheel name="right_back_wheel"  x="-0.15" y="-0.17"/>
-<xacro:wheel name="left_front_wheel"  x="0.15" y="0.17"/>
-<xacro:wheel name="left_back_wheel"   x="-0.15" y="0.17"/>
-</robot>
+/home/miko/mobile_robot_ws/src/my_robot_description/urdf/mobile_robot.urdf.xacro

File: src/my_robot_description/urdf/mobile_robot.urdf.xacro (robot description, xacro)
@@ -6,4 +6,13 @@
   <xacro:property name="wheellen" value="0.1" />
   <xacro:property name="wheeldia" value="0.07" />
+<xacro:macro name="default_inertial" params="mass">
+  <inertial>
+    <mass value="${mass}"/>
+    <inertia
+      ixx="0.01" ixy="0.0" ixz="0.0"
+      iyy="0.01" iyz="0.0"
+      izz="0.01"/>
+  </inertial>
+</xacro:macro>
   <material name="blue">
     <color rgba="0 0 0.8 1"/>
@@ -22,4 +31,10 @@
     <material name="blue"/>
   </visual>
+  <collision>
+    <geometry>
+      <box size="${length} ${width} ${height}"/>
+    </geometry>
+  </collision>
+  <xacro:default_inertial mass="5.0"/>
   </link>
   <xacro:macro name="wheel" params="name x y">
@@ -32,4 +47,11 @@
         <material name="black"/>
       </visual>
+       <collision>
+    <origin rpy="1.57075 0 0" xyz="0 0 0"/>
+    <geometry>
+      <cylinder length="${wheellen}" radius="${wheeldia/2}"/>
+    </geometry>
+  </collision>
+  <xacro:default_inertial mass="0.5"/>
     </link>
      <joint name="$base_to_${name}" type="fixed">
