Commit message: Made joints continuous for  model

File: src/my_robot_description/urdf/mobile_robot.urdf.xacro (robot description, xacro)
@@ -55,5 +55,5 @@
   <xacro:default_inertial mass="0.5"/>
     </link>
-     <joint name="$base_to_${name}" type="fixed">
+     <joint name="$base_to_${name}" type="continuous">
       <axis xyz="0 1 0" rpy="0 0 0" />
       <parent link="base_link"/>

Commit message: Made the robot controllable Gazebo

File: src/my_robot_description/urdf/mobile_robot.urdf.xacro (robot description, xacro)
@@ -6,4 +6,19 @@
   <xacro:property name="wheellen" value="0.1" />
   <xacro:property name="wheeldia" value="0.07" />
+  <ros2_control name="GazeboSystem" type="system">
+  <hardware>
+    <plugin>gazebo_ros2_control/GazeboSystem</plugin>
+  </hardware>
+  <joint name="left_front_wheel_joint">
+    <command_interface name="velocity"/>
+    <state_interface name="position"/>
+    <state_interface name="velocity"/>
+  </joint>
+  <joint name="right_front_wheel_joint">
+    <command_interface name="velocity"/>
+    <state_interface name="position"/>
+    <state_interface name="velocity"/>
+  </joint>
+</ros2_control>
 <xacro:macro name="default_inertial" params="mass">
   <inertial>
@@ -55,5 +70,5 @@
   <xacro:default_inertial mass="0.5"/>
     </link>
-     <joint name="$base_to_${name}" type="continuous">
+     <joint name="${name}_joint" type="continuous">
       <axis xyz="0 1 0" rpy="0 0 0" />
       <parent link="base_link"/>
@@ -66,3 +81,8 @@
 <xacro:wheel name="left_front_wheel"  x="0.15" y="0.17"/>
 <xacro:wheel name="left_back_wheel"   x="-0.15" y="0.17"/>
+<gazebo>
+  <plugin name="gazebo_ros2_control" filename="libgazebo_ros2_control.so">
+    <parameters>/home/miko/mobile_robot_ws/install/my_robot_description/share/my_robot_description/config/controllers.yaml</parameters>
+  </plugin>
+</gazebo>
 </robot>

Commit message: Tried Implementing SLAM but still not perfect

File: src/my_robot_description/urdf/mobile_robot.urdf.xacro (robot description, xacro)
@@ -1,4 +1,4 @@
 <?xml version="1.0"?>
-<robot name="macroed" xmlns:xacro="http://ros.org/wiki/xacro">
+<robot name="macroed" xmlns:xacro="http://www.ros.org/wiki/xacro">
   <xacro:include filename="$(find my_robot_description)/urdf/sensors/lidar.xacro"/>
   <xacro:include filename="$(find my_robot_description)/urdf/sensors/camera.xacro"/>
@@ -9,27 +9,58 @@
   <xacro:property name="wheeldia" value="0.07" />
   <ros2_control name="GazeboSystem" type="system">
-  <hardware>
-    <plugin>gazebo_ros2_control/GazeboSystem</plugin>
-  </hardware>
-  <joint name="left_front_wheel_joint">
-    <command_interface name="velocity"/>
-    <state_interface name="position"/>
-    <state_interface name="velocity"/>
-  </joint>
-  <joint name="right_front_wheel_joint">
-    <command_interface name="velocity"/>
-    <state_interface name="position"/>
-    <state_interface name="velocity"/>
-  </joint>
-</ros2_control>
-<xacro:macro name="default_inertial" params="mass">
-  <inertial>
-    <mass value="${mass}"/>
-    <inertia
-      ixx="0.01" ixy="0.0" ixz="0.0"
-      iyy="0.01" iyz="0.0"
-      izz="0.01"/>
-  </inertial>
-</xacro:macro>
+    <hardware>
+      <plugin>gazebo_ros2_control/GazeboSystem</plugin>
+    </hardware>
+    <joint name="left_front_wheel_joint">
+      <command_interface name="velocity"/>
+      <state_interface name="position"/>
+      <state_interface name="velocity"/>
+    </joint>
+    <joint name="left_back_wheel_joint">
+      <command_interface name="velocity"/>
+      <state_interface name="position"/>
+      <state_interface name="velocity"/>
+    </joint>
+    <joint name="right_front_wheel_joint">
+      <command_interface name="velocity"/>
+      <state_interface name="position"/>
+      <state_interface name="velocity"/>
+    </joint>
+    <joint name="right_back_wheel_joint">
+      <command_interface name="velocity"/>
+      <state_interface name="position"/>
+      <state_interface name="velocity"/>
+    </joint>
+  </ros2_control>
+  <!-- INERTIAL MACROS -->
+  <xacro:macro name="default_inertial" params="mass">
+    <inertial>
+      <mass value="${mass}"/>
+      <inertia
+        ixx="0.01" ixy="0.0" ixz="0.0"
+        iyy="0.01" iyz="0.0"
+        izz="0.01"/>
+    </inertial>
+  </xacro:macro>
+  <xacro:macro name="base_inertial" params="mass">
+    <inertial>
+      <origin xyz="0 0 -0.03" rpy="0 0 0"/>
+      <mass value="${mass}"/>
+      <inertia
+        ixx="0.03" ixy="0.0" ixz="0.0"
+        iyy="0.03" iyz="0.0"
+        izz="0.05"/>
+    </inertial>
+  </xacro:macro>
+  <!-- correct cylinder inertia for wheels -->
+  <xacro:macro name="wheel_inertial" params="mass">
+    <inertial>
+      <mass value="${mass}"/>
+      <inertia
+        ixx="0.001" ixy="0.0" ixz="0.0"
+        iyy="0.001" iyz="0.0"
+        izz="0.0005"/>
+    </inertial>
+  </xacro:macro>
   <material name="blue">
     <color rgba="0 0 0.8 1"/>
@@ -41,22 +72,40 @@
     <color rgba="1 1 1 1"/>
   </material>
-   <link name="base_link">
-  <visual>
-    <geometry>
-     <box size="${length} ${width} ${height}"/>
-    </geometry>
-    <material name="blue"/>
-  </visual>
-  <collision>
-    <geometry>
-      <box size="${length} ${width} ${height}"/>
-    </geometry>
-  </collision>
-  <xacro:default_inertial mass="5.0"/>
+  <!-- BASE LINK -->
+  <link name="base_link">
+    <visual>
+      <geometry>
+        <box size="${length} ${width} ${height}"/>
+      </geometry>
+      <material name="blue"/>
+    </visual>
+    <visual>
+      <origin xyz="0 0 0.02" rpy="0 0 0"/>
+      <geometry>
+        <box size="0.48 0.48 0.12"/>
+      </geometry>
+      <material name="white"/>
+    </visual>
+    <!-- collision matches smaller visual, stays within wheelbase -->
+    <collision>
+      <geometry>
+        <box size="${length} ${width} ${height}"/>
+      </geometry>
+    </collision>
+    <!-- reduced mass for more realistic physics -->
+    <xacro:default_inertial mass="3.0"/>
   </link>
+  <!-- after the closing </link> of base_link, before WHEEL MACRO -->
+<gazebo reference="base_link">
+    <mu1>0.5</mu1>
+    <mu2>0.5</mu2>
+    <kp>100000.0</kp>
+    <kd>10.0</kd>
+</gazebo>
+  <!-- WHEEL MACRO -->
   <xacro:macro name="wheel" params="name x y">
     <link name="${name}">
       <visual>
-        <origin xyz="0 0 0" rpy="${pi/2} 0 0" />
+        <origin xyz="0 0 0" rpy="${pi/2} 0 0"/>
         <geometry>
           <cylinder radius="${wheeldia/2}" length="${wheellen}"/>
@@ -64,35 +113,46 @@
         <material name="black"/>
       </visual>
-       <collision>
-    <origin rpy="1.57075 0 0" xyz="0 0 0"/>
-    <geometry>
-      <cylinder length="${wheellen}" radius="${wheeldia/2}"/>
-    </geometry>
-  </collision>
-  <xacro:default_inertial mass="0.5"/>
+      <collision>
+        <origin xyz="0 0 0" rpy="${pi/2} 0 0"/>
+        <geometry>
+          <cylinder radius="${wheeldia/2}" length="${wheellen}"/>
+        </geometry>
+      </collision>
+      <!-- correct cylinder inertia -->
+      <xacro:wheel_inertial mass="0.5"/>
     </link>
-     <joint name="${name}_joint" type="continuous">
-      <axis xyz="0 1 0" rpy="0 0 0" />
+    <joint name="${name}_joint" type="continuous">
+      <axis xyz="0 1 0"/>
       <parent link="base_link"/>
       <child link="${name}"/>
       <origin xyz="${x} ${y} -0.05" rpy="0 0 0"/>
     </joint>
+    <!-- balanced friction and contact params -->
+    <gazebo reference="${name}">
+      <mu1>2.0</mu1>
+      <mu2>2.0</mu2>
+      <kp>100000.0</kp>
+      <kd>10.0</kd>
+    </gazebo>
   </xacro:macro>
-   <xacro:lidar_sensor
+  <!-- SENSORS -->
+  <xacro:lidar_sensor
     parent_link="base_link"
     xyz="0.15 0 0.12"
     rpy="0 0 0"/>
-    <xacro:camera_sensor
-  parent_link="base_link"
-  xyz="0.20 0 0.14"
-  rpy="0 0 0"/>
-<xacro:wheel name="right_front_wheel" x="0.15" y="-0.17"/>
-<xacro:wheel name="right_back_wheel"  x="-0.15" y="-0.17"/>
-<xacro:wheel name="left_front_wheel"  x="0.15" y="0.17"/>
-<xacro:wheel name="left_back_wheel"   x="-0.15" y="0.17"/>
-<gazebo>
-  <plugin name="gazebo_ros2_control" filename="libgazebo_ros2_control.so">
-    <parameters>/home/miko/mobile_robot_ws/install/my_robot_description/share/my_robot_description/config/controllers.yaml</parameters>
-  </plugin>
-</gazebo>
+  <xacro:camera_sensor
+    parent_link="base_link"
+    xyz="0.20 0 0.14"
+    rpy="0 0 0"/>
+  <!-- WHEELS -->
+  <xacro:wheel name="right_front_wheel" x="0.15"  y="-0.17"/>
+  <xacro:wheel name="right_back_wheel"  x="-0.15" y="-0.17"/>
+  <xacro:wheel name="left_front_wheel"  x="0.15"  y="0.17"/>
+  <xacro:wheel name="left_back_wheel"   x="-0.15" y="0.17"/>
+  <!-- GAZEBO ROS2 CONTROL PLUGIN -->
+  <gazebo>
+    <plugin name="gazebo_ros2_control" filename="libgazebo_ros2_control.so">
+      <parameters>/home/miko/mobile_robot_ws/install/my_robot_description/share/my_robot_description/config/controllers.yaml</parameters>
+    </plugin>
+  </gazebo>
 </robot>

File: src/my_robot_description/urdf/sensors/lidar.xacro (robot description, xacro)
@@ -62,5 +62,5 @@
         <plugin name="gazebo_ros_lidar_controller" filename="libgazebo_ros_ray_sensor.so">
           <ros>
-            <remapping>~/out:=scan</remapping>
+            <remapping>~/out:=/scan</remapping>
           </ros>
           <output_type>sensor_msgs/LaserScan</output_type>
